Commit message: changed chassis and drive wheels in apjr.gazebo to fix contacts (Moi and Tata). Changed nav params with ref to diffbot github, and replaced DWA Planner with Teb local planner which is more suited for car like robots, now no more in place rotation and collisions

File: apjr_bringup/robot_description/urdf/apjr_backup.xacro (robot description, xacro)
@@ -66,8 +66,8 @@
         <collision>
             <xacro:driveWheel_geometry/>
-            <surface>
+            <!-- <surface>
                 <friction>
                     <ode>
-                    <mu>0</mu>
+                    <mu>0.5</mu>
                     <mu2>0</mu2>
                     <slip1>0.0</slip1>
@@ -81,9 +81,9 @@
                     </ode>
                 </contact>
-            </surface>
+            </surface>    -->
         </collision>
     </link>
     <xacro:wheel_joint parent="chassis" child="right_chassis_caster_wheel" offset="${-chassisLength/2 + 0.05} ${-chassisWidth/2 - wheelWidth/2}  ${-chassisHeight/2 - wheelRadius}" axis="0 1 0"/>
-    <xacro:wheel_transmission wheel="right_chassis_caster_wheel"/>
+    <!-- <xacro:wheel_transmission wheel="right_chassis_caster_wheel"/> -->
          <!-- ################################### Right Fork Caster Wheel link #####################################-->
     <!-- <link name="left_chassis_caster_wheel">
@@ -122,5 +122,5 @@
         <collision>
             <xacro:driveWheel_geometry/>
-            <surface>
+            <!-- <surface>
                 <friction>
                     <ode>
@@ -134,12 +134,12 @@
                     <ode>
                     <kp>1e15</kp>
-                    <kd>1e13</kd>
+                    <kd>100</kd>
                     </ode>
                 </contact>
-            </surface>
+            </surface>    -->
         </collision>
     </link>
     <xacro:wheel_joint parent="chassis" child="left_chassis_caster_wheel" offset="${-chassisLength/2 + 0.05} ${chassisWidth/2 + wheelWidth/2}  ${-chassisHeight/2 - wheelRadius}" axis="0 1 0"/>
-    <xacro:wheel_transmission wheel="left_chassis_caster_wheel"/>
+    <!-- <xacro:wheel_transmission wheel="left_chassis_caster_wheel"/> -->
     <!-- ################################### Right Fork Link #####################################-->
     <link name="fork_right">
@@ -160,5 +160,5 @@
     <xacro:fixed_offset_joint parent="chassis" child="fork_right" offset="${chassisLength/2 + forkLength/2} ${-chassisWidth/2 + forkWidth/2} ${-chassisHeight/2 + forkHeight/2}"/>
         <!-- ################################### Right Fork Caster Wheel link #####################################-->
-    <link name="right_fork_caster_wheel">
+    <!-- <link name="right_fork_caster_wheel">
         <inertial>
             <xacro:casterWheel_inertial/>
@@ -169,17 +169,7 @@
         <collision name="right_fork_caster_wheel">
             <xacro:casterWheel_geometry/>
-            <surface>
-            <friction>
-                <ode>
-                <mu>0</mu>
-                <mu2>0</mu2>
-                <slip1>0.0</slip1>
-                <slip2>0.0</slip2>
-                </ode>
-            </friction>
-            </surface>
-        </collision>
-    </link>
-    <xacro:wheel_joint parent="chassis" child="right_fork_caster_wheel" offset="${chassisLength/2 + forkLength/2 + 0.2} ${-chassisWidth/2 + forkWidth/2} ${-chassisHeight/2 + casterRadius -wheelRadius*2}" axis="0 1 0"/>
+        </collision>
+    </link>
+    <xacro:wheel_joint parent="chassis" child="right_fork_caster_wheel" offset="${chassisLength/2 + forkLength/2 + 0.2} ${-chassisWidth/2 + forkWidth/2} ${-chassisHeight/2 + casterRadius -wheelRadius*2}" axis="0 1 0"/> -->
     <!-- ################################### Left Fork Link #####################################-->
     <link name="fork_left">
@@ -199,6 +189,6 @@
     </link>
     <xacro:fixed_offset_joint parent="chassis" child="fork_left" offset="${chassisLength/2 + forkLength/2} ${chassisWidth/2 - forkWidth/2} ${-chassisHeight/2 + forkHeight/2}"/>
-    <!-- ################################### Left Fork Caster Wheel link #####################################-->
-    <link name="left_fork_caster_wheel">
+    ################################### Left Fork Caster Wheel link #####################################
+    <!-- <link name="left_fork_caster_wheel">
         <inertial>
             <xacro:casterWheel_inertial/>
@@ -209,17 +199,7 @@
         <collision name="left_fork_caster_wheel">
             <xacro:casterWheel_geometry/>
-            <surface>
-            <friction>
-                <ode>
-                <mu>0</mu>
-                <mu2>0</mu2>
-                <slip1>1.0</slip1>
-                <slip2>1.0</slip2>
-                </ode>
-            </friction>
-            </surface>
-        </collision>
-    </link>
-    <xacro:wheel_joint parent="chassis" child="left_fork_caster_wheel" offset="${chassisLength/2 + forkLength/2 + 0.2} ${chassisWidth/2 - forkWidth/2} ${-chassisHeight/2 + casterRadius -wheelRadius*2}" axis="0 1 0"/>
+        </collision>
+    </link>
+    <xacro:wheel_joint parent="chassis" child="left_fork_caster_wheel" offset="${chassisLength/2 + forkLength/2 + 0.2} ${chassisWidth/2 - forkWidth/2} ${-chassisHeight/2 + casterRadius -wheelRadius*2}" axis="0 1 0"/>  -->
     <!-- ################################### Shaft link #####################################-->
     	<!-- <link name="drive_wheel_shaft">
@@ -310,5 +290,5 @@
         <collision>
             <xacro:driveWheel_geometry/>
-            <surface>
+            <!-- <surface>
                 <friction>
                     <ode>
@@ -325,5 +305,5 @@
                     </ode>
                 </contact>
-            </surface>
+            </surface>    -->
         </collision>
     </link>
@@ -343,5 +323,5 @@
         <collision>
             <xacro:driveWheel_geometry/>
-            <surface>
+            <!-- <surface>
                 <friction>
                     <ode>
@@ -358,5 +338,5 @@
                     </ode>
                 </contact>
-            </surface>
+            </surface>    -->
         </collision>
     </link>
