Commit message: add new changes

File: apjr_bringup/robot_description/urdf/apjr.xacro (robot description, xacro)
@@ -31,5 +31,5 @@
     <xacro:fixed_offset_joint parent="base_footprint" child="chassis" offset="0 0 ${chassisHeight/2 + 0.16}"/>
      <!-- ################################### Right Fork Caster Wheel link #####################################-->
-    <link name="right_chassis_caster_wheel">
+    <!-- <link name="right_chassis_caster_wheel">
         <inertial>
             <xacro:casterWheel_inertial/>
@@ -52,7 +52,39 @@
         </collision>
     </link>
-    <xacro:wheel_joint parent="chassis" child="right_chassis_caster_wheel" offset="0.0 ${-chassisWidth/2 + forkWidth/2} ${-chassisHeight/2 + casterRadius -wheelRadius*2}" axis="0 1 0"/>
+    <xacro:wheel_joint parent="chassis" child="right_chassis_caster_wheel" offset="0.0 ${-chassisWidth/2 + forkWidth/2} ${-chassisHeight/2 + casterRadius -wheelRadius*2}" axis="0 1 0"/> -->
+    <link name="right_chassis_caster_wheel">
+        <inertial>
+            <xacro:driveWheel_inertial/>
+        </inertial>
+        <visual name="right_chassis_caster_wheel">
+            <xacro:driveWheel_geometry/>
+            <material name="">
+                <color rgba="0.3 1.0 0.0 1.0"/>
+                <texture filename=""/>
+            </material>
+        </visual>
+        <collision>
+            <xacro:driveWheel_geometry/>
+            <surface>
+                <friction>
+                    <ode>
+                    <mu>0</mu>
+                    <mu2>0</mu2>
+                    <slip1>0.0</slip1>
+                    <slip2>0.0</slip2>
+                    </ode>
+                </friction>
+                <contact>
+                    <ode>
+                    <kp>1e15</kp>
+                    <kd>1e13</kd>
+                    </ode>
+                </contact>
+            </surface>
+        </collision>
+    </link>
+    <xacro:wheel_joint parent="chassis" child="right_chassis_caster_wheel" offset="${-chassisLength/2 + 0.05} ${-chassisWidth/2 - wheelWidth/2}  ${-chassisHeight/2 - wheelRadius}" axis="0 1 0"/>
          <!-- ################################### Right Fork Caster Wheel link #####################################-->
-    <link name="left_chassis_caster_wheel">
+    <!-- <link name="left_chassis_caster_wheel">
         <inertial>
             <xacro:casterWheel_inertial/>
@@ -75,5 +107,37 @@
         </collision>
     </link>
-    <xacro:wheel_joint parent="chassis" child="left_chassis_caster_wheel" offset="0.0 ${chassisWidth/2 - forkWidth/2} ${-chassisHeight/2 + casterRadius -wheelRadius*2}" axis="0 1 0"/>
+    <xacro:wheel_joint parent="chassis" child="left_chassis_caster_wheel" offset="0.0 ${chassisWidth/2 - forkWidth/2} ${-chassisHeight/2 + casterRadius -wheelRadius*2}" axis="0 1 0"/> -->
+        <link name="left_chassis_caster_wheel">
+        <inertial>
+            <xacro:driveWheel_inertial/>
+        </inertial>
+        <visual name="left_chassis_caster_wheel">
+            <xacro:driveWheel_geometry/>
+            <material name="">
+                <color rgba="0.3 1.0 0.0 1.0"/>
+                <texture filename=""/>
+            </material>
+        </visual>
+        <collision>
+            <xacro:driveWheel_geometry/>
+            <surface>
+                <friction>
+                    <ode>
+                    <mu>0</mu>
+                    <mu2>0</mu2>
+                    <slip1>0.0</slip1>
+                    <slip2>0.0</slip2>
+                    </ode>
+                </friction>
+                <contact>
+                    <ode>
+                    <kp>1e15</kp>
+                    <kd>1e13</kd>
+                    </ode>
+                </contact>
+            </surface>
+        </collision>
+    </link>
+    <xacro:wheel_joint parent="chassis" child="left_chassis_caster_wheel" offset="${-chassisLength/2 + 0.05} ${chassisWidth/2 + wheelWidth/2}  ${-chassisHeight/2 - wheelRadius}" axis="0 1 0"/>
     <!-- ################################### Right Fork Link #####################################-->
     <link name="fork_right">
@@ -171,14 +235,33 @@
 	<!-- <xacro:fixed_offset_joint parent="chassis" child="drive_wheel_shaft" offset="0.0 0.0 ${-chassisHeight/2 - wheelRadius}"/> -->
     <!-- ################################### Hinge link #####################################-->
-    <link name="drive_wheel_hinge">
+    <!-- <link name="drive_wheel_hinge">
 		<visual>
-			<!-- <material name="white"/> -->
+			 <material name="white"/>
 			<xacro:hinge_geometry/>
 		</visual>
-		<!--<collision>
+		<<collision>
 			<xacro:hinge_geometry/>
-		</collision>-->
+		</collision>
 		<inertial>
-			<!-- <xacro:hinge_inertial/> -->
+			<xacro:hinge_inertial/>
+            <mass value="0.05" />
+		<inertia ixx="0"
+			 ixy="0"
+			 ixz="0"
+			 iyy="0"
+			 iyz="0"
+			 izz="${2/5*0.05*(0.015*0.015)}"
+		/>
+		</inertial>
+	</link>
+    <link name="drive_wheel_right_hinge">
+		<visual>
+			<xacro:hinge_geometry/>
+		</visual>
+		<collision>
+			<xacro:hinge_geometry/>
+		</collision>
+		<inertial>
+			<xacro:hinge_inertial/>
             <mass value="0.05" />
 		<inertia ixx="0"
@@ -192,5 +275,5 @@
 	</link>
     <joint name="steering_joint" type="revolute">
-        <origin xyz="0.0 0.0 ${-chassisHeight/2 - wheelRadius}" rpy="0 0 0"/>
+        <origin xyz="${chassisLength/2 - 0.05} ${chassisWidth/2 + wheelWidth/2}  ${-chassisHeight/2 - wheelRadius}" rpy="0 0 0"/>
         <parent link="chassis"/>
         <child link="drive_wheel_hinge"/>
@@ -200,6 +283,15 @@
         <dynamics damping="1" friction="0"/>
     </joint>
-	<!-- <xacro:hinge_joint parent="chassis" child="drive_wheel_hinge" offset="0.0 0.0 ${-chassisHeight/2 - wheelRadius}"/> -->
+    <joint name="steering_right_joint" type="revolute">
+        <origin xyz="${chassisLength/2 - 0.05} ${-chassisWidth/2 - wheelWidth/2}  ${-chassisHeight/2 - wheelRadius}" rpy="0 0 0"/>
+        <parent link="chassis"/>
+        <child link="drive_wheel_right_hinge"/>
+        <axis xyz="0 0 1"/>
+        <limit lower="-1.570796" upper="1.570796" effort="1000000" velocity="100"/>
+        <joint_properties damping="1.0" friction="1.0"/>
+        <dynamics damping="1" friction="0"/>
+    </joint>
 	<xacro:hinge_transmission hinge="steering"/>
+    <xacro:hinge_transmission hinge="steering_right"/> -->
     <!-- ################################### Drive Wheel link #####################################-->
     <link name="drive_wheel">
@@ -235,16 +327,55 @@
     </link>
 	<xacro:wheel_transmission wheel="drive_wheel"/>
+        <!-- ################################### Drive Wheel Right link #####################################-->
+    <link name="drive_wheel_right">
+        <inertial>
+            <xacro:driveWheel_inertial/>
+        </inertial>
+        <visual name="drive_wheel_right">
+            <xacro:driveWheel_geometry/>
+            <material name="">
+                <color rgba="0.3 1.0 0.0 1.0"/>
+                <texture filename=""/>
+            </material>
+        </visual>
+        <collision>
+            <xacro:driveWheel_geometry/>
+            <surface>
+                <friction>
+                    <ode>
+                    <mu>0</mu>
+                    <mu2>0</mu2>
+                    <slip1>0.0</slip1>
+                    <slip2>0.0</slip2>
+                    </ode>
+                </friction>
+                <contact>
+                    <ode>
+                    <kp>1e15</kp>
+                    <kd>1e13</kd>
+                    </ode>
+                </contact>
+            </surface>
+        </collision>
+    </link>
+	<xacro:wheel_transmission wheel="drive_wheel_right"/>
     <!-- ################################### Joints #####################################-->
     <joint name="drive_wheel_joint" type="continuous">
-        <origin xyz="0.0 0.0 0.0" rpy="0.0 0.0 0.0"/>
+        <!-- <origin xyz="0.0 0.0 0.0" rpy="0.0 0.0 0.0"/> -->
+        <origin xyz="${chassisLength/2 - 0.05} ${chassisWidth/2 + wheelWidth/2}  ${-chassisHeight/2 - wheelRadius}" rpy="0 0 0"/>
         <!-- <origin xyz="0.0 0.0 ${-chassisHeight/2 - wheelRadius} " rpy="0.0 0.0 0.0"/> -->
-        <parent link="drive_wheel_hinge"/>
+        <!-- <parent link="drive_wheel_hinge"/> -->
+        <parent link="chassis"/>
         <child link="drive_wheel"/>
         <axis xyz="0.0 1.0 0.0"/>
-       <!-- <limit lower="0" upper="0.0" effort="1000000" velocity="1000.0"/>
-       <joint_properties damping="0.5" friction="1"/> -->
-        <!-- <limit lower="0" upper="0" effort="10" velocity="1000.0"/>
-       <joint_properties damping="1.0" friction="1.0"/>
-       <dynamics damping="1" friction="0"/> -->
+    </joint>
+    <joint name="drive_wheel_right_joint" type="continuous">
+        <!-- <origin xyz="0.0 0.0 0.0" rpy="0.0 0.0 0.0"/> -->
+        <origin xyz="${chassisLength/2 - 0.05} ${-chassisWidth/2 - wheelWidth/2}  ${-chassisHeight/2 - wheelRadius}" rpy="0 0 0"/>
+        <!-- <origin xyz="0.0 0.0 ${-chassisHeight/2 - wheelRadius} " rpy="0.0 0.0 0.0"/> -->
+        <!-- <parent link="drive_wheel_right_hinge"/> -->
+        <parent link="chassis"/>
+        <child link="drive_wheel_right"/>
+        <axis xyz="0.0 1.0 0.0"/>
     </joint>
     <!-- ################################### base_scan Link #####################################-->

File: apjr_bringup/robot_description/urdf/physicalProperties.xacro (robot description, xacro)
@@ -1,18 +1,18 @@
 <?xml version="1.0"?>
 <robot xmlns:xacro="http://ros.org/wiki/xacro" name="apjr">
-    <xacro:property name="chassisHeight" value="0.7"/>
-    <xacro:property name="chassisLength" value="0.5"/>
-    <xacro:property name="chassisWidth" value="0.5"/>
+    <xacro:property name="chassisHeight" value="0.4"/>
+    <xacro:property name="chassisLength" value=".365"/>
+    <xacro:property name="chassisWidth" value="0.475"/>
     <xacro:property name="chassisMass" value="40"/>
     <xacro:property name="forkHeight" value="0.1"/>
-    <xacro:property name="forkLength" value="0.8"/>
-    <xacro:property name="forkWidth" value="0.15"/>
+    <xacro:property name="forkLength" value="0.55"/>
+    <xacro:property name="forkWidth" value="0.11"/>
     <xacro:property name="forkMass" value="10"/>
     <xacro:property name="casterRadius" value="0.05"/>
     <xacro:property name="casterMass" value="3"/>
-    <xacro:property name="wheelWidth" value="0.05"/>
-    <xacro:property name="wheelRadius" value="0.08"/>
+    <xacro:property name="wheelWidth" value="0.03"/>
+    <xacro:property name="wheelRadius" value="0.05"/>
     <xacro:property name="wheelPos" value="0.2"/>
-    <xacro:property name="wheelMass" value="10"/>
+    <xacro:property name="wheelMass" value="1"/>
     <!-- Chassis -->
 	<xacro:macro name="chassis_geometry">

Commit message: added pallet model

File: apjr_bringup/robot_description/urdf/apjr.xacro (robot description, xacro)
@@ -412,3 +412,23 @@
 </joint>
   <link name="imu_link"/>
+<!-- ################################### Camera  #####################################-->
+  <joint name="camera_joint" type="fixed">
+    <origin xyz="${chassisLength/2} 0.0 ${chassisHeight}" rpy="0 0.5236 0"/>
+    <parent link="chassis"/>
+    <child link="camera_link"/>
+  </joint>
+  <link name="camera_link">
+    <collision>
+      <origin xyz="0.0 0.0 0.0" rpy="0 0 0"/>
+      <geometry>
+        <box size="0.01 0.01 0.01"/>
+      </geometry>
+    </collision>
+    <visual>
+      <origin xyz="0 0 0" rpy="0 0 0"/>
+      <geometry>
+            <box size="0.01 0.01 0.01"/>
+      </geometry>
+      </visual>
+  </link>
 </robot>

Commit message: odom, lidar, gmapping, nav all working real life

File: apjr_bringup/robot_description/urdf/apjr.xacro (robot description, xacro)
@@ -382,5 +382,6 @@
     </joint>
     <!-- ################################### base_scan Link #####################################-->
-    <link name="base_scan">
+    <!-- was base_scan -->
+    <link name="laser">
     <collision>
       <origin xyz="0 0 0" rpy="0 0 0"/>
@@ -406,5 +407,5 @@
         <origin xyz="0 0 ${chassisHeight/2 + 0.05}" rpy="0 0 0"/>
         <parent link="chassis"/>
-        <child link="base_scan"/>
+        <child link="laser"/>
     </joint>
 <joint name="imu_joint" type="fixed">
